File: Miniscope-v4-Wire-Free-KiCad/KiCad/Miniscope-v4-Wire-Free/Miniscope-v4-Wire-Free.kicad_pcb (KiCad board)
At the start: 6 copper layers, 26.7 x 12.2 mm, 117 parts, among them J1 0475710001, J10 Conn_01x01, J11 Conn_01x01, J12 Conn_01x01, J14 Conn_01x01, J15 Conn_01x01, J16 Conn_01x01, J17 Conn_01x01, J18 Conn_01x01, J19 Conn_01x01, J2 Conn_01x04, J20 Conn_01x01, J21 Conn_01x01, J22 Conn_01x01, J23 Conn_01x01, J24 Conn_01x01, J25 Conn_01x01, J26 Conn_01x01, J27 Conn_01x01, J3 Conn_01x04, J4 Conn_01x01, J5 Conn_01x01, J6 Conn_01x01, J7 Conn_01x01, J8 Conn_01x01, J9 Conn_01x01, Q1 NTK3134NT1G, Q2 MMBT3904LP-7B, SW1 TL3780AF330QG, U1 LTC3554, U2 HV892, U3 LTC3218, U4 MAX13030EETE+BGA, U5 TSOP57438TT1, U6 ATSAMD51J20A-UUT-EFP, U7 NCP163AMX330TBG, U8 NOIP1SN0480A, U9 LMV321IDCKR, Y2 Crystal

Commit message: My Miniscope-v4-Wire-Free Fork
- components with new fields: MPN & OEPS PN
- almost all components with these new fields filled in
- some still missing: waiting new codes to be emitted
Parts:
- D2, D3: value LED_Small_ALT -> LTST-C191KEKT
- J10, J11, J12, J14, J15, J16, J17, J18, J19, J20, J21, J22, J23, J24, J25, J26, J27, J4, J5, J6, J7, J8, J9: value Conn_01x01 -> DNP
- J2: value Conn_01x04 -> DNP
- L3: value L_Small -> BLM18PG471SN1D
- R1, R17: value 25K -> 24.9k
- R12: value DNL -> DNP
- R13: value 400K -> 402k
- R15: value 37K -> 37.4k
- R18: value R_Small_US -> 1k8
- R3: value 1.25M -> 1.27M
- R6: value 649K -> 649k
- R7, R8: value 2.2K -> 2.2k
- R9: value 8.2K -> 8.2k
- U4: value MAX13030EETE+BGA -> MAX13030EEBE+T
- U6: value ATSAMD51J20A-UUT-EFP -> ATSAMD51J20A
- U8: value NOIP1SN0480A -> NOIP1SN0480A-STI
- Y2: value Crystal -> XTAL 32.7680KHZ
