File: Miniscope-v4-Wire-Free-KiCad/KiCad/Miniscope-v4-Wire-Free/Miniscope-v4-Wire-Free.kicad_sch (KiCad schematic)
At the start: 115 parts, among them J1 0475710001, J10 Conn_01x01, J11 Conn_01x01, J12 Conn_01x01, J14 Conn_01x01, J15 Conn_01x01, J16 Conn_01x01, J17 Conn_01x01, J18 Conn_01x01, J19 Conn_01x01, J2 Conn_01x04, J20 Conn_01x01, J21 Conn_01x01, J22 Conn_01x01, J23 Conn_01x01, J24 Conn_01x01, J25 Conn_01x01, J26 Conn_01x01, J27 Conn_01x01, J3 Conn_01x04, J4 Conn_01x01, J5 Conn_01x01, J6 Conn_01x01, J7 Conn_01x01, J8 Conn_01x01, J9 Conn_01x01, Q1 NTK3134NT1G, Q2 MMBT3904LP-7B, SW1 TL3780AF330QG, U1 LTC3554, U2 HV892, U3 LTC3218, U4 MAX13030EETE+BGA, U5 TSOP57438TT1, U6 ATSAMD51J20A-UUT-EFP, U7 NCP163AMX330TBG, U8 NOIP1SN0480A, U9 LMV321IDCKR, Y2 Crystal

Commit message: My Miniscope-v4-Wire-Free Fork
- components with new fields: MPN & OEPS PN
- almost all components with these new fields filled in
- some still missing: waiting new codes to be emitted
Parts:
- C1, C2, C26, C35, C50, C51, C52, C6, C7: MPN (none) -> CL05A106MP5NUNC; OEPS PN (none) -> OEPS010038
- C10, C19, C22, C23, C24, C25, C27, C28, C30, C38, C40, C41, C42, C43, C44, C45, C46, C47, C48, C49, C53, C9: MPN (none) -> GRM033R61E104KE14J; OEPS PN (none) -> OEPS010035
- C11, C12, C13, C15, C5: MPN (none) -> CM03X5R225M10AH; OEPS PN (none) -> OEPS010042
- C14, C37: MPN (none) -> CL03A105MO3NRNH; OEPS PN (none) -> OEPS010036
- C16: MPN (none) -> 885012206112; OEPS PN (none) -> OEPS010014
- C17, C29, C36: MPN (none) -> GRM035R60J475ME15D; OEPS PN (none) -> TBD
- C18, C20: MPN (none) -> GRM0335C1H270GA01D; OEPS PN (none) -> OEPS010029
- C3, C4: MPN (none) -> GRM0335C1H100JA01J; OEPS PN (none) -> OEPS010060
- D1: MPN (none) -> LXZ1-PR01; OEPS PN (none) -> OEPS030021
- D2, D3: value LED_Small_ALT -> LTST-C191KEKT; MPN (none) -> LTST-C191KEKT; OEPS PN (none) -> TBD
- J1: MPN (none) -> 0475710001; OEPS PN (none) -> TBD
- J10, J11, J12, J14, J15, J16, J17, J18, J19, J20, J21, J22, J23, J24, J25, J26, J27, J4, J5, J6, J7, J8, J9: value Conn_01x01 -> DNP; MPN (none) -> n.a.; OEPS PN (none) -> n.a.
- J2: value Conn_01x04 -> DNP; MPN (none) -> n.a.; OEPS PN (none) -> n.a.
- J3: MPN (none) -> FH19C-4S-0.5SH(10); OEPS PN (none) -> TBD
- L1, L5: MPN (none) -> MLZ1608N100LT000; OEPS PN (none) -> TBD
- L2: MPN (none) -> !! CIG21L4R7MNE Obsolete; to select a new one; OEPS PN (none) -> TBD !! OEPS040017 Obsolete
- L3: value L_Small -> BLM18PG471SN1D; MPN (none) -> BLM18PG471SN1D; OEPS PN (none) -> OEPS040014
- L4: MPN (none) -> BLM18PG471SN1D; OEPS PN (none) -> OEPS040014
- Q1: MPN (none) -> NTK3134NT1G; OEPS PN (none) -> TBD
- Q2: MPN (none) -> MMBT3904LP-7B; OEPS PN (none) -> OEPS060014
- R1, R17: value 25K -> 24.9k; MPN (none) -> CRCW020124K9FNED; OEPS PN (none) -> TBD
- R10: MPN (none) -> RC0201FR-072KL; OEPS PN (none) -> OEPS020067
- R11, R19: MPN (none) -> RC0201FR-071KL; OEPS PN (none) -> OEPS020065
- R12: value DNL -> DNP; MPN (none) -> n.a.; OEPS PN (none) -> n.a.
- R13: value 400K -> 402k; MPN (none) -> ERJ-1GNF4023C; OEPS PN (none) -> TBD
- R14, R16, R20: MPN (none) -> ERJ-1GNF1003C; OEPS PN (none) -> OEPS020072
- R15: value 37K -> 37.4k; MPN (none) -> ERJ-1GNF3742C; OEPS PN (none) -> TBD
- R18: value R_Small_US -> 1k8; MPN (none) -> ERJ-1GNF1801C; OEPS PN (none) -> TBD
- R2: MPN (none) -> ERJ-1GNF1801C; OEPS PN (none) -> OEPS020074
- R21: renamed from R?; MPN (none) -> ERJ-1GNF1002C; OEPS PN (none) -> OEPS020071
- R22: renamed from R?; MPN (none) -> ERJ-1GNF4752C; OEPS PN (none) -> OEPS020075
- R3: value 1.25M -> 1.27M; MPN (none) -> CRCW02011M27FNED; OEPS PN (none) -> TBD
- R4: MPN (none) -> CRCW02012M05FNED; OEPS PN (none) -> TBD
- R5: MPN (none) -> CRCW02011M00FNED; OEPS PN (none) -> TBD
- R6: value 649K -> 649k; MPN (none) -> RC0201FR-07649KL; OEPS PN (none) -> TBD
- R7, R8: value 2.2K -> 2.2k; MPN (none) -> RC0201FR-072K2L; OEPS PN (none) -> TBD
- R9: value 8.2K -> 8.2k; MPN (none) -> ERJ-1GNF8201C; OEPS PN (none) -> TBD
- SW1: MPN (none) -> TL3780AF330QG; OEPS PN (none) -> TBD
- U1: MPN (none) -> LTC3554EUD#PBF; OEPS PN (none) -> TBD
- U2: MPN (none) -> HV892K7-G; OEPS PN (none) -> TBD
- U3: MPN (none) -> LTC3218EDDB#TRMPBF; OEPS PN (none) -> OEPS080069
- U4: value MAX13030EETE+BGA -> MAX13030EEBE+T; MPN (none) -> MAX13030EEBE+T; OEPS PN (none) -> TBD
- U5: MPN (none) -> TSOP57438TT1; OEPS PN (none) -> OEPSJ1008
- U6: value ATSAMD51J20A-UUT-EFP -> ATSAMD51J20A; MPN (none) -> ATSAMD51J20A-UUT-EFP; OEPS PN (none) -> TBD
- U7: MPN (none) -> NCP163AMX330TBG; OEPS PN (none) -> OEPS080076
- U8: value NOIP1SN0480A -> NOIP1SN0480A-STI; MPN (none) -> NOIP1SN0480A-STI; OEPS PN (none) -> TBD
- U9: MPN (none) -> LMV321IDCKR; OEPS PN (none) -> OEPS080068
- Y2: value Crystal -> XTAL 32.7680KHZ; MPN (none) -> 9HT11-32.768KBZF-T; OEPS PN (none) -> TBD

Commit message: final v4
Parts:
- C17, C29, C36: OEPS PN TBD -> OEPS010065
- D2, D3: OEPS PN TBD -> OEPS030029
- J1: OEPS PN TBD -> OEPS070078
- J3: OEPS PN TBD -> OEPS070077
- L1, L5: OEPS PN TBD -> OEPS040021
- L2: MPN !! CIG21L4R7MNE Obsolete; to select a new one -> MLP2012S4R7MT0S1; OEPS PN TBD !! OEPS040017 Obsolete -> OEPS040022
- Q1: OEPS PN TBD -> OEPS060015
- R1, R17: OEPS PN TBD -> OEPS020105
- R13: OEPS PN TBD -> OEPS020112
- R15: OEPS PN TBD -> OEPS020113
- R18: OEPS PN TBD -> OEPS020114
- R3: OEPS PN TBD -> OEPS020106
- R4: OEPS PN TBD -> OEPS020107
- R5: OEPS PN TBD -> OEPS020108
- R6: OEPS PN TBD -> OEPS020109
- R7, R8: OEPS PN TBD -> OEPS020110
- R9: OEPS PN TBD -> OEPS020111
- SW1: OEPS PN TBD -> OEPS100050
- U1: OEPS PN TBD -> OEPS080113
- U2: OEPS PN TBD -> OEPS080111
- U4: OEPS PN TBD -> OEPS080114
- U5: OEPS PN OEPSJ1008 -> OEPS080117
- U6: OEPS PN TBD -> OEPS080115
- U8: value NOIP1SN0480A-STI -> NOIP1SP0480A-STI; MPN NOIP1SN0480A-STI -> NOIP1SP0480A-STI; OEPS PN TBD -> OEPS080071
- Y2: OEPS PN TBD -> OEPS100051
